File: systems/systems_interface_pcb/tvac_systems_interface.sch (EAGLE design)
At the start: 6 parts, among them J1 171-025-213R001, J2 A-DS09A/KG-T2S, J3 A-DS09A/KG-T2S, J4 A-DS09A/KG-T2S, X1 TERMINAL-BLOCK-3.5MM-6-PIN-RO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

Commit message: Add files via upload
hand-routed using Jaden and Lorna's advice
Connections:
- net +3V3: now also J2.2; no longer J3.9
- net +5V: now also J2.1; no longer J2.2
- net +BAT: now also J2.8, J2.9; no longer J4.1, J4.2
- net CANH: now also J2.3; no longer J2.7
- net CANL: now also J4.2; no longer J2.9
- net DIS_TRANS_UARTN: now also J2.5; no longer J2.4
- net PAY_MOSI_A/TX: now also J3.9; no longer J2.1
- net PAY_RST: now also J2.4; no longer J2.5
- net PAY_SCK_A/TX: now also J2.7; no longer J2.3
- net RTC_VBATT: now also J4.1; no longer J2.8
